Commit message: update tf launch

File: src/direct_lidar_odometry/urdf/m2_test.urdf (robot description, URDF)
Before this commit: robot m2d, 12 links, 11 joints
Links:
- link base_link: geometry collision box size=1.66 0.9 0.55; visual mesh filename=package://direct_lidar_odometry/models/M2_P.stl scale=0.001 0.001 0.001
